Commit message: Bugfixing and fine tuning FR3

File: configs/pybullet/envs/assets/franka_panda/fr3.urdf (robot description, URDF)
Before this commit: robot fr3, 17 links, 16 joints
Links:
- removed link fr3_link0_sc
- removed link fr3_link1_sc
- removed link fr3_link2_sc
- removed link fr3_link3_sc
- removed link fr3_link4_sc
- removed link fr3_link5_sc
- removed link fr3_link6_sc
- removed link fr3_link7_sc
- removed link fr3_link8
- link fr3_link0: mass None -> 0.629769
- link fr3_link1: mass None -> 4.970684
- link fr3_link2: mass None -> 0.646926
- link fr3_link3: mass None -> 3.228604
- link fr3_link4: mass None -> 3.587895
- link fr3_link5: mass None -> 1.225946
- link fr3_link6: mass None -> 1.666555
- link fr3_link7: mass None -> 0.735522
Joints:
- removed joint fr3_joint8
- removed joint fr3_link0_sc_joint
- removed joint fr3_link1_sc_joint
- removed joint fr3_link2_sc_joint
- removed joint fr3_link3_sc_joint
- removed joint fr3_link4_sc_joint
- removed joint fr3_link5_sc_joint
- removed joint fr3_link6_sc_joint
- removed joint fr3_link7_sc_joint

File: configs/pybullet/envs/assets/franka_panda/fr3_hand.urdf (robot description, URDF)
Before this commit: robot fr3, 22 links, 21 joints
Links:
- removed link fr3_hand_sc
- removed link fr3_hand_tcp
- removed link fr3_link0_sc
- removed link fr3_link1_sc
- removed link fr3_link2_sc
- removed link fr3_link3_sc
- removed link fr3_link4_sc
- removed link fr3_link5_sc
- removed link fr3_link6_sc
- removed link fr3_link7_sc
- removed link fr3_link8
- link fr3_hand: mass None -> 0.73
- link fr3_leftfinger: mass None -> 0.015
- link fr3_link0: mass None -> 0.629769
- link fr3_link1: mass None -> 4.970684
- link fr3_link2: mass None -> 0.646926
- link fr3_link3: mass None -> 3.228604
- link fr3_link4: mass None -> 3.587895
- link fr3_link5: mass None -> 1.225946
- link fr3_link6: mass None -> 1.666555
- link fr3_link7: mass None -> 0.735522
- link fr3_rightfinger: mass None -> 0.015
Joints:
- removed joint fr3_hand_sc_joint
- removed joint fr3_hand_tcp_joint
- removed joint fr3_joint8
- removed joint fr3_link0_sc_joint
- removed joint fr3_link1_sc_joint
- removed joint fr3_link2_sc_joint
- removed joint fr3_link3_sc_joint
- removed joint fr3_link4_sc_joint
- removed joint fr3_link5_sc_joint
- removed joint fr3_link6_sc_joint
- removed joint fr3_link7_sc_joint
- joint fr3_hand_joint: origin xyz=0 0 0 rpy=0 0 -0.7853981633974483 -> xyz=0 0 0.107 rpy=0 0 -0.7853981633974483; parent fr3_link8 -> fr3_link7
